Commit message: comment gravity

File: engix_description/urdf/engix.urdf (robot description, URDF)
Before this commit: robot engix, 19 links, 18 joints
Links:
- link caster_left: mass 0.3 -> 0.1
- link caster_right: mass 0.3 -> 0.1
- link caster_wheel_left: mass 0.5 -> 0.4
- link caster_wheel_right: mass 0.5 -> 0.4
- link lwheel: mass 2.5 -> 4.0
- link rwheel: mass 2.5 -> 4.0
Joints:
- removed joint ZED2
- removed joint battery
- removed joint dc_dc
- removed joint jetson_nano
- removed joint lan
- removed joint left_wheel
- removed joint lidar_tof
- removed joint right_wheel
- removed joint usb_hub
- added joint ZED2_joint: type fixed, parent base_link, child ZED2_1, origin xyz=0.176645 0.00992 0.4957 rpy=0 0 0
- added joint battery__joint: type fixed, parent base_link, child battery_1, origin xyz=0.011102 0.015765 0.1077 rpy=0 0 0
- added joint dc_dc_joint: type fixed, parent base_link, child dc_dc_1, origin xyz=0.027645 -0.10808 0.2157 rpy=0 0 0
- added joint jetson_nano_joint: type fixed, parent base_link, child jetson_nano_1, origin xyz=-0.02108 0.10192 0.21904 rpy=0 0 0
- added joint lan_joint: type fixed, parent base_link, child lan_1, origin xyz=0.07857 0.10192 0.2157 rpy=0 0 0
- added joint left_wheel_joint: type continuous, parent base_link, child lwheel, origin xyz=-0.133355 0.150817 0.079162 rpy=0 0 0, axis 0.0 1.0 -0.0
- added joint lidar_tof_joint: type fixed, parent base_link, child lidar_tof_1, origin xyz=0.157645 -0.04512 0.3677 rpy=0 0 0
- added joint right_wheel_joint: type continuous, parent base_link, child rwheel, origin xyz=-0.133355 -0.146183 0.079162 rpy=0 0 0, axis 0.0 1.0 -0.0
- added joint usb_hub_joint: type fixed, parent base_link, child usb_hub_1, origin xyz=-0.077355 0.00192 0.3177 rpy=0 0 0

Commit message: delete launcher move_base node and fix urdf model

File: engix_description/urdf/engix.urdf (robot description, URDF)
Before this commit: robot engix, 19 links, 18 joints
Links:
- link caster_left: mass 0.1 -> 0.3
- link caster_right: mass 0.1 -> 0.3
- link caster_wheel_left: mass 0.4 -> 0.5
- link caster_wheel_right: mass 0.4 -> 0.5
- link lwheel: mass 4.0 -> 2.5
- link rwheel: mass 4.0 -> 2.5
Joints:
- removed joint battery__joint
- removed joint left_wheel_joint
- removed joint right_wheel_joint
- added joint battery_joint: type fixed, parent base_link, child battery_1, origin xyz=0.011102 0.015765 0.1077 rpy=0 0 0
- added joint left_wheel: type continuous, parent base_link, child lwheel, origin xyz=-0.133355 0.150817 0.079162 rpy=0 0 0, axis 0.0 1.0 -0.0
- added joint right_wheel: type continuous, parent base_link, child rwheel, origin xyz=-0.133355 -0.146183 0.079162 rpy=0 0 0, axis 0.0 1.0 -0.0

Commit message: other fix

File: engix_description/urdf/engix.urdf (robot description, URDF)
Before this commit: robot engix, 19 links, 18 joints
Links:
- link lidar_tof_1: geometry visual mesh filename=package://engix_description/meshes/lidar_tof_1.stl scale=0.001 0.001 0.001

Commit message: add rgbd camera

File: engix_description/urdf/engix.urdf (robot description, URDF)
Before this commit: robot engix, 19 links, 18 joints
Links:
- added link camera_depth_frame, mass 0.001
- added link camera_depth_optical_frame, mass 0.001
- added link camera_link, mass 0.001
- added link camera_rgb_frame, mass 0.001
- added link camera_rgb_optical_frame, mass 0.001
Joints:
- added joint camera_depth_joint: type fixed, parent camera_rgb_frame, child camera_depth_frame, origin xyz=0.176645 0.00992 0.4957 rpy=0 0 0
- added joint camera_depth_optical_joint: type fixed, parent camera_depth_frame, child camera_depth_optical_frame, origin xyz=0.176645 0.00992 0.4957 rpy=0 0 0
- added joint camera_joint: type fixed, parent camera_rgb_frame, child camera_link, origin xyz=0.176645 0.00992 0.4957 rpy=0 0 0
- added joint camera_rgb_joint: type fixed, parent base_link, child camera_rgb_frame, origin xyz=0.176645 0.00992 0.4957 rpy=0 0 0
- added joint camera_rgb_optical_joint: type fixed, parent camera_rgb_frame, child camera_rgb_optical_frame, origin xyz=0.176645 0.00992 0.4957 rpy=0 0 0

Commit message: poind cloud fix view axis

File: engix_description/urdf/engix.urdf (robot description, URDF)
Before this commit: robot engix, 24 links, 23 joints
Links:
- link camera_depth_frame: mass 0.001 -> None
- link camera_depth_optical_frame: mass 0.001 -> None
- link camera_rgb_optical_frame: mass 0.001 -> None
Joints:
- joint camera_depth_optical_joint: origin xyz=0.176645 0.00992 0.4957 rpy=0 0 0 -> xyz=0.176645 0.00992 0.4957 rpy=-1.5707 0 -1.5707

Commit message: add tof-fov lidar

File: engix_description/urdf/engix.urdf (robot description, URDF)
Before this commit: robot engix, 24 links, 23 joints
Links:
- removed link lidar_tof_1
- added link lidar_tof; visual mesh filename=package://engix_description/meshes/lidar_tof_1.stl scale=0.001 0.001 0.001
Joints:
- joint lidar_tof_joint: child lidar_tof_1 -> lidar_tof

Commit message: fix tof_lidar, lidar message pointcloud2

File: engix_description/urdf/engix.urdf (robot description, URDF)
Before this commit: robot engix, 24 links, 23 joints
Links:
- removed link lidar_tof
- added link laser_tof; collision mesh filename=package://engix_description/meshes/lidar_tof_1.stl scale=0.001 0.001 0.001; visual mesh filename=package://engix_description/meshes/lidar_tof_1.stl scale=0.001 0.001 0.001
Joints:
- removed joint lidar_tof_joint
- added joint laser_tof_joint: type fixed, parent base_link, child laser_tof, origin xyz=0.157645 -0.04512 0.3677 rpy=0 0 0

Commit message: diff_repair

File: engix_description/urdf/engix.urdf (robot description, URDF)
Before this commit: robot engix, 24 links, 23 joints
Joints:
- removed joint left_wheel
- removed joint right_wheel
- added joint left_wheel_joint: type continuous, parent base_link, child lwheel, origin xyz=-0.133355 0.150817 0.079162 rpy=0 0 0, axis 0.0 1.0 -0.0
- added joint right_wheel_joint: type continuous, parent base_link, child rwheel, origin xyz=-0.133355 -0.146183 0.079162 rpy=0 0 0, axis 0.0 1.0 -0.0

Commit message: big update, add odrive can driver

File: engix_description/urdf/engix.urdf (robot description, URDF)
Before this commit: robot engix, 24 links, 23 joints
Links:
- removed link ZED2_1
- removed link battery_1
- removed link camera_depth_frame
- removed link camera_depth_optical_frame
- removed link camera_link
- removed link camera_rgb_frame
- removed link camera_rgb_optical_frame
- removed link dc_dc_1
- removed link gps_1
- removed link jetson_nano_1
- removed link lan_1
- removed link laser_tof
- removed link usb_hub_1
- added link battery; collision mesh filename=package://engix_description/meshes/battery.STL; visual mesh filename=package://engix_description/meshes/battery.STL
- added link cover, mass 0.1; collision mesh filename=package://engix_description/meshes/cover.STL; visual mesh filename=package://engix_description/meshes/cover.STL
- added link deck; collision mesh filename=package://engix_description/meshes/deck.STL; visual mesh filename=package://engix_description/meshes/deck.STL
- added link gps; collision mesh filename=package://engix_description/meshes/gps.STL; visual mesh filename=package://engix_description/meshes/gps.STL
- added link stop; collision mesh filename=package://engix_description/meshes/stop.STL; visual mesh filename=package://engix_description/meshes/stop.STL
- added link ultrasound_center; collision mesh filename=package://engix_description/meshes/ultrasound_center.STL
- added link ultrasound_left_back
- added link ultrasound_left_back_back
- added link ultrasound_left_top
- added link ultrasound_right_back
- added link ultrasound_right_back_back
- added link ultrasound_right_top
- added link zed; collision mesh filename=package://engix_description/meshes/zed.STL; visual mesh filename=package://engix_description/meshes/zed.STL
- link base_link: geometry collision mesh filename=package://engix_description/meshes/base_link.STL; visual mesh filename=package://engix_description/meshes/base_link.STL
- link caster_left: mass 0.3 -> 1.0; geometry collision mesh filename=package://engix_description/meshes/caster_left.STL; visual mesh filename=package://engix_description/meshes/caster_left.STL
- link caster_right: mass 0.3 -> 1.0; geometry collision mesh filename=package://engix_description/meshes/caster_right.STL; visual mesh filename=package://engix_description/meshes/caster_right.STL
- link caster_wheel_left: mass 0.5 -> 1.0; geometry collision mesh filename=package://engix_description/meshes/caster_wheel_left.STL; visual mesh filename=package://engix_description/meshes/caster_wheel_left.STL
- link caster_wheel_right: mass 0.5 -> 1.0; geometry collision mesh filename=package://engix_description/meshes/caster_wheel_right.STL; visual mesh filename=package://engix_description/meshes/caster_wheel_right.STL
- link inertial_link: mass 15.034 -> 10
- link laser: geometry collision mesh filename=package://engix_description/meshes/laser.STL; visual mesh filename=package://engix_description/meshes/laser.STL
- link lwheel: mass 2.5 -> 4.637; geometry collision mesh filename=package://engix_description/meshes/lwheel.STL; visual mesh filename=package://engix_description/meshes/lwheel.STL
- link rwheel: mass 2.5 -> 4.637; geometry collision mesh filename=package://engix_description/meshes/rwheel.STL; visual mesh filename=package://engix_description/meshes/rwheel.STL
Joints:
- removed joint ZED2_joint
- removed joint camera_depth_joint
- removed joint camera_depth_optical_joint
- removed joint camera_joint
- removed joint camera_rgb_joint
- removed joint camera_rgb_optical_joint
- removed joint caster_left_joint
- removed joint dc_dc_joint
- removed joint jetson_nano_joint
- removed joint lan_joint
- removed joint laser_tof_joint
- removed joint left_wheel_joint
- removed joint right_wheel_joint
- removed joint rp_laser_joint
- removed joint usb_hub_joint
- added joint caster_left: type continuous, parent base_link, child caster_left, origin xyz=0.643 0.39037 0.091717 rpy=0 0 0, axis 0 0 1
- added joint cover_joint: type fixed, parent base_link, child cover, origin xyz=-0.162 -0.0044742 -0.016717 rpy=0 0 3.1416, axis 0 0 0
- added joint deck_joint: type fixed, parent base_link, child deck, origin xyz=0 0 0 rpy=0 0 0, axis 0 0 0
- added joint laser_joint: type fixed, parent base_link, child laser, origin xyz=-0.056018 -0.0047765 0.48823 rpy=0 0 0, axis 0 0 0
- added joint left_wheel: type continuous, parent base_link, child lwheel, origin xyz=-0.59511 0.42022 -0.11179 rpy=0 0 0, axis 0 1 -1.3832E-05
- added joint right_wheel: type continuous, parent base_link, child rwheel, origin xyz=-0.59511 -0.42022 -0.11179 rpy=0 0 0, axis 0 1 -1.3832E-05
- added joint stop_joint: type fixed, parent base_link, child stop, origin xyz=-0.69 -0.37937 0.40441 rpy=0 0 0, axis 0 0 0
- added joint ultrasound_center_joint: type fixed, parent base_link, child ultrasound_center, origin xyz=0.67838 -0.00040907 0.10435 rpy=0 0 0, axis 0 0 0
- added joint ultrasound_left_back_back_joint: type fixed, parent base_link, child ultrasound_left_back_back, origin xyz=-0.8798 0.19399 -0.05687 rpy=0 0 -3.25, axis 0 0 0
- added joint ultrasound_left_back_joint: type fixed, parent base_link, child ultrasound_left_back, origin xyz=-0.66119 0.37242 0.27466 rpy=0 0 -4.7, axis 0 0 0
- added joint ultrasound_left_top_joint: type fixed, parent base_link, child ultrasound_left_top, origin xyz=0.41729 0.33052 -0.0062646 rpy=0 0 -4.7, axis 0 0 0
- added joint ultrasound_right_back_back_joint: type fixed, parent base_link, child ultrasound_right_back_back, origin xyz=-0.8798 -0.20253 -0.05687 rpy=0 0 -3, axis 0 0 0
- added joint ultrasound_right_back_joint: type fixed, parent base_link, child ultrasound_right_back, origin xyz=-0.66113 -0.37937 0.27466 rpy=0 0 -1.5708, axis 0 0 0
- added joint ultrasound_right_top_joint: type fixed, parent base_link, child ultrasound_right_top, origin xyz=0.41736 -0.33598 -0.0062646 rpy=0 0 -1.5708, axis 0 0 0
- added joint zed_joint: type fixed, parent base_link, child zed, origin xyz=-0.064262 -0.0023649 0.54982 rpy=0 0 0, axis 0 0 0
- joint battery_joint: axis (none) -> 0 0 0; child battery_1 -> battery; origin xyz=0.011102 0.015765 0.1077 rpy=0 0 0 -> xyz=-0.63961 -0.098618 -0.044982 rpy=1.5708 0 -3.1416
- joint caster_right_joint: axis 0.0 0.0 -1.0 -> 0 0 1; origin xyz=0.155465 -0.084832 0.072019 rpy=0 0 0 -> xyz=0.643 -0.39932 0.091717 rpy=0 0 0
- joint caster_wheel_left_joint: axis -0.0 -1.0 0.0 -> 0 1 0; origin xyz=-0.016 -0.0025 -0.046 rpy=0 0 0 -> xyz=0.067678 0 -0.27618 rpy=0 0 0
- joint caster_wheel_right_joint: axis -0.0 -1.0 0.0 -> 0 1 0; origin xyz=-0.016 -0.0025 -0.046 rpy=0 0 0 -> xyz=0.067678 0 -0.27618 rpy=0 0 0
- joint gps_joint: axis (none) -> 0 0 0; child gps_1 -> gps; origin xyz=0.112558 -0.00808 0.4957 rpy=0 0 0 -> xyz=-0.079471 0.11632 0.54778 rpy=0 0 0
- joint imu_joint: axis (none) -> 0 0 0; origin xyz=0.176645 0.00992 0.4957 rpy=0 0 0 -> xyz=-0.064262 -0.0023649 0.54982 rpy=0 0 0

Commit message: update configs

File: engix_description/urdf/engix.urdf (robot description, URDF)
Before this commit: robot engix, 24 links, 23 joints
Joints:
- joint ultrasound_center_joint: origin xyz=0.67838 -0.00040907 0.10435 rpy=0 0 0 -> xyz=0.58 -0.00040907 0.10435 rpy=0 0 0
